File: rc13-mbed-main-board.sch (EAGLE design)
At the start: 54 parts, among them IC1 MBED_MICROCONTROLLER, U1 PCA9555PW,118, X1 BALL_SENS, X2 ETH, X5 BTNS, X9 COIL

Commit message: Routed some board
Parts:
- removed LED3, LED4, LED5: (no value), led:LEDCHIP-LED0603
- removed R31, R32, R33, R34, R8: 2K2, rcl:R-EU_R0603
Connections:
- removed net LED2: R7.2
- removed net LED3: R8.2
- removed net LED4: R33.2
- removed net LED5: R34.2, U1.IO1_7
- removed net N$10: LED_5V.A, R15.2
- removed net N$11: LED4.A, R33.1
- removed net N$12: LED5.A, R34.1
- removed net N$15: R15.1
- removed net SCL2: IC1.P$27, R32.1
- removed net SDA2: IC1.P$28, R31.1
- net +3V3: now also LED1.A; no longer R31.2, R32.2
- net +5V: now also R15.2
- net BALL: now also IC1.P$28
- net CHARGE: now also IC1.P$20; no longer IC1.P$19
- net GND: now also LED_5V.A; no longer LED1.C, LED3.C, LED4.C, LED5.C
- net KICK: now also IC1.P$19; no longer IC1.P$20
- net LED1: now also R7.2, U1.IO1_7
- net N$7: now also LED1.C; no longer LED1.A
- net N$9: now also LED_5V.C, R15.1; no longer LED3.A, R8.1
Other:
- moved on the sheet: LED1, LED_5V, R15, R17

Commit message: Some routing changes
Parts:
- removed C3, C4: 470uF, rcl:CPOL-EUE3.5-8
Connections:
- net +15V: no longer C3.+, C4.+
- net GND: no longer C3.-, C4.-
Changed lines of the file:
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@@
 <part name="C1" library="rcl" deviceset="C-EU" device="C0603K" value="100nF"/>
 <part name="C2" library="rcl" deviceset="CPOL-EU" device="E3.5-8" value="470uF"/>
-<part name="C3" library="rcl" deviceset="CPOL-EU" device="E3.5-8" value="470uF"/>
-<part name="C4" library="rcl" deviceset="CPOL-EU" device="E3.5-8" value="470uF"/>
 <part name="C9" library="rcl" deviceset="CPOL-EU" device="E3.5-8" value="470uF"/>
 <part name="LED_5V" library="led" deviceset="LED" device="CHIP-LED0603"/>
@@
 <instance part="C1" gate="G$1" x="48.26" y="127"/>
 <instance part="C2" gate="G$1" x="187.96" y="124.46"/>
-<instance part="C3" gate="G$1" x="198.12" y="124.46"/>
-<instance part="C4" gate="G$1" x="208.28" y="124.46"/>
 <instance part="C9" gate="G$1" x="177.8" y="124.46"/>
 <instance part="LED_5V" gate="G$1" x="208.28" y="142.24" rot="R180"/>
@@
 <wire x1="187.96" y1="116.84" x2="177.8" y2="116.84" width="0.1524" layer="91"/>
 <wire x1="177.8" y1="116.84" x2="167.64" y2="116.84" width="0.1524" layer="91"/>
-<wire x1="187.96" y1="116.84" x2="198.12" y2="116.84" width="0.1524" layer="91"/>
-<pinref part="C3" gate="G$1" pin="-"/>
-<wire x1="198.12" y1="116.84" x2="198.12" y2="119.38" width="0.1524" layer="91"/>
-<wire x1="198.12" y1="116.84" x2="208.28" y2="116.84" width="0.1524" layer="91"/>
-<pinref part="C4" gate="G$1" pin="-"/>
-<wire x1="208.28" y1="116.84" x2="208.28" y2="119.38" width="0.1524" layer="91"/>
 <junction x="167.64" y="116.84"/>
-<junction x="187.96" y="116.84"/>
-<junction x="198.12" y="116.84"/>
 <pinref part="C9" gate="G$1" pin="-"/>
 <wire x1="177.8" y1="116.84" x2="177.8" y2="119.38" width="0.1524" layer="91"/>
@@
 </segment>
 <segment>
-<wire x1="208.28" y1="129.54" x2="198.12" y2="129.54" width="0.1524" layer="91"/>
-<wire x1="198.12" y1="129.54" x2="187.96" y2="129.54" width="0.1524" layer="91"/>
 <wire x1="187.96" y1="129.54" x2="177.8" y2="129.54" width="0.1524" layer="91"/>
 <wire x1="177.8" y1="129.54" x2="167.64" y2="129.54" width="0.1524" layer="91"/>
@@
 <pinref part="C2" gate="G$1" pin="+"/>
 <wire x1="187.96" y1="127" x2="187.96" y2="129.54" width="0.1524" layer="91"/>
-<pinref part="C3" gate="G$1" pin="+"/>
-<wire x1="198.12" y1="127" x2="198.12" y2="129.54" width="0.1524" layer="91"/>
-<pinref part="C4" gate="G$1" pin="+"/>
-<wire x1="208.28" y1="127" x2="208.28" y2="129.54" width="0.1524" layer="91"/>
-<junction x="187.96" y="129.54"/>
-<junction x="198.12" y="129.54"/>
 <pinref part="C9" gate="G$1" pin="+"/>
 <wire x1="177.8" y1="127" x2="177.8" y2="129.54" width="0.1524" layer="91"/>
