File: rc13-mbed-main-board2.sch (EAGLE design)
At the start: 44 parts, among them IC1 MBED_MICROCONTROLLER, U1 PCA9555PW,118, X1 BALL_SENS, X2 ETH, X5 BTNS, X9 COIL

Commit message: Few small changes
Parts:
- added C3: 470uF, rcl:CPOL-EUE3.5-8
Connections:
- net +15V: now also C3.+
- net GND: now also C3.-
Changed lines of the file:
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@@
 <part name="P+8" library="supply1" deviceset="+5V" device=""/>
 <part name="GND15" library="supply1" deviceset="GND" device=""/>
+<part name="C3" library="rcl" deviceset="CPOL-EU" device="E3.5-8" value="470uF"/>
 </parts>
 <sheets>
@@
 <instance part="P+8" gate="1" x="208.28" y="165.1"/>
 <instance part="GND15" gate="1" x="208.28" y="134.62"/>
+<instance part="C3" gate="G$1" x="198.12" y="124.46"/>
 </instances>
 <busses>
@@
 <junction x="177.8" y="116.84"/>
 <pinref part="GND16" gate="1" pin="GND"/>
+<pinref part="C3" gate="G$1" pin="-"/>
+<wire x1="198.12" y1="119.38" x2="198.12" y2="116.84" width="0.1524" layer="91"/>
+<wire x1="198.12" y1="116.84" x2="187.96" y2="116.84" width="0.1524" layer="91"/>
+<junction x="187.96" y="116.84"/>
 </segment>
 <segment>
@@
 <junction x="137.16" y="129.54"/>
 <pinref part="BAT_15V" gate="G$1" pin="P$1"/>
-</segment>
-</net>
+<pinref part="C3" gate="G$1" pin="+"/>
+<wire x1="198.12" y1="127" x2="198.12" y2="129.54" width="0.1524" layer="91"/>
+<wire x1="198.12" y1="129.54" x2="187.96" y2="129.54" width="0.1524" layer="91"/>
+<junction x="187.96" y="129.54"/>
+</segment>
+</net>
